Commit message: tested with Gazebo

File: seer_description/urdf/seer_robot_base.urdf.xacro (robot description, xacro)
@@ -16,14 +16,14 @@
   <link name="base_link">
     <visual>
-      <origin xyz="0 0 0.2" rpy="0 0 0" />
+      <origin xyz="0 0 0.21" rpy="0 0 0" />
       <geometry>
         <mesh filename="package://seer_description/meshes/robot_body.stl" scale="0.1 0.1 0.1" />
       </geometry>
-      <material name="white">
-        <color rgba="0.9 0.9 0.9 1.0" />
+      <material name="orange">
+        <color rgba="0.922 0.57 0.82 1.0" />
       </material>
     </visual>
     <collision>
-      <origin xyz="0 0 0.15" rpy="0 0 0" />
+      <origin xyz="0 0 0.2" rpy="0 0 0" />
       <geometry>
         <box size="0.8 0.5 0.3" />
@@ -149,23 +149,3 @@
     </plugin>
   </gazebo>
-  <!-- <gazebo>
-    <plugin name="gazebo_ros_diff_drive" filename="libgazebo_ros_diff_drive.so">
-      <ros>
-        <namespace>/</namespace>
-        <remapping>cmd_vel:=cmd_vel</remapping>
-        <remapping>odom:=odom</remapping>
-      </ros>
-      <left_joint>left_wheel_joint</left_joint>
-      <right_joint>right_wheel_joint</right_joint>
-      <wheel_separation>${wheel_ygap * 2}</wheel_separation>
-      <wheel_diameter>${wheel_radius * 2}</wheel_diameter>
-      <max_wheel_torque>200</max_wheel_torque>
-      <max_wheel_acceleration>10.0</max_wheel_acceleration>
-      <publish_odom>true</publish_odom>
-      <publish_odom_tf>true</publish_odom_tf>
-      <publish_wheel_tf>true</publish_wheel_tf>
-      <odometry_frame>odom</odometry_frame>
-      <robot_base_frame>base_footprint</robot_base_frame>
-    </plugin>
-  </gazebo> -->
 </robot>

Commit message: update for gazebo simulation and rviz

File: seer_description/urdf/seer_robot_base.urdf.xacro (robot description, xacro)
@@ -7,5 +7,5 @@
   <xacro:property name="wheel_ygap" value="0.3" />
   <xacro:property name="wheel_xoff" value="0.0" />
-  <xacro:property name="wheel_zoff" value="0.05" />
+  <xacro:property name="wheel_zoff" value="0.1" />
   <link name="base_footprint" />
   <joint name="base_joint" type="fixed">
@@ -16,5 +16,5 @@
   <link name="base_link">
     <visual>
-      <origin xyz="0 0 0.21" rpy="0 0 0" />
+      <origin xyz="0 0 0.26" rpy="0 0 ${pi}" />
       <geometry>
         <mesh filename="package://seer_description/meshes/robot_body.stl" scale="0.1 0.1 0.1" />
@@ -32,6 +32,5 @@
     <inertial>
       <origin xyz="0 0 0.15" rpy="0 0 0" />
-      <mass value="${base_mass}" />
-      <inertia ixx="1.0" ixy="0.0" ixz="0.0" iyy="1.0" iyz="0.0" izz="1.0" />
+      <mass value="${base_mass}" /> <inertia ixx="3.11" ixy="0.0" ixz="0.0" iyy="6.68" iyz="0.0" izz="8.15" />
     </inertial>
   </link>
@@ -68,4 +67,35 @@
   <xacro:drive_wheel prefix="left" y_reflect="1" filename="left_wheel.stl" />
   <xacro:drive_wheel prefix="right" y_reflect="-1" filename="right_wheel.stl" />
+  <xacro:macro name="lidar" params="prefix xy_reflect x_offset y_offset filename">
+    <link name="${prefix}_lidar_link">
+      <visual>
+        <origin xyz="0 0 0" rpy="0 0 0" />
+        <geometry>
+          <mesh filename="package://seer_description/meshes/${filename}" scale="0.1 0.1 0.1" />
+        </geometry>
+        <material name="grey">
+          <color rgba="0.5 0.5 0.5 1.0" />
+        </material>
+      </visual>
+      <collision>
+        <origin xyz="0 0 0" rpy="0 0 0" />
+        <geometry>
+          <cylinder radius="0.05" length="0.08"  />
+        </geometry>
+      </collision>
+      <inertial>
+        <origin xyz="0 0 0" rpy="0 0 0" />
+        <mass value="0.3" />
+        <inertia ixx="0.01" ixy="0.0" ixz="0.0" iyy="0.01" iyz="0.0" izz="0.01" />
+      </inertial>
+    </link>
+    <joint name="${prefix}_lidar_joint" type="fixed">
+      <parent link="base_link" />
+      <child link="${prefix}_lidar_link" />
+      <origin xyz="${x_offset*xy_reflect} ${y_offset*xy_reflect} 0.15" rpy="0 0 0" />
+    </joint>
+  </xacro:macro>
+  <xacro:lidar prefix="front" xy_reflect="1" x_offset="0.38" y_offset="0.25" filename="lidar.stl" />
+  <xacro:lidar prefix="back" xy_reflect="-1" x_offset="0.38" y_offset="0.25" filename="lidar.stl" />
   <link name="front_caster">
     <collision>
@@ -80,9 +110,9 @@
     </inertial>
   </link>
-  <joint name="front_caster_joint" type="fixed">
+  <!-- <joint name="front_caster_joint" type="fixed">
     <parent link="base_link" />
     <child link="front_caster" />
     <origin xyz="0.3 0 ${wheel_zoff}" rpy="0 0 0" />
-  </joint>
+  </joint> -->
   <link name="rear_caster">
     <collision>
@@ -97,8 +127,18 @@
     </inertial>
   </link>
+  <!-- <joint name="rear_caster_joint" type="fixed">
+    <parent link="base_link" />
+    <child link="rear_caster" />
+    <origin xyz="-0.3 0 ${wheel_zoff}" rpy="0 0 0" />
+  </joint> -->
+  <joint name="front_caster_joint" type="fixed">
+    <parent link="base_link" />
+    <child link="front_caster" />
+    <origin xyz="0.3 0 ${wheel_radius - 0.005}" rpy="0 0 0" />
+  </joint>
   <joint name="rear_caster_joint" type="fixed">
     <parent link="base_link" />
     <child link="rear_caster" />
-    <origin xyz="-0.3 0 ${wheel_zoff}" rpy="0 0 0" />
+    <origin xyz="-0.3 0 ${wheel_radius - 0.005}" rpy="0 0 0" />
   </joint>
   <!-- control simulation gazebo -->
