Commit message: update for lidar simulation in gazebo

File: seer_description/urdf/seer_robot_base.urdf (robot description, URDF)
Before this commit: robot seer_amb, 6 links, 5 joints
Links:
- added link back_lidar_link, mass 0.3; collision cylinder length=0.08 radius=0.05; visual mesh filename=package://seer_description/meshes/lidar.stl scale=0.1 0.1 0.1
- added link front_lidar_link, mass 0.3; collision cylinder length=0.08 radius=0.05; visual mesh filename=package://seer_description/meshes/lidar.stl scale=0.1 0.1 0.1
Joints:
- added joint back_lidar_joint: type fixed, parent base_link, child back_lidar_link, origin xyz=-0.38 -0.25 0.15 rpy=0 0 0
- added joint front_lidar_joint: type fixed, parent base_link, child front_lidar_link, origin xyz=0.38 0.25 0.15 rpy=0 0 0
- joint base_joint: origin xyz=0.0 0.0 0.05 rpy=0 0 0 -> xyz=0.0 0.0 0.0 rpy=0 0 0
- joint front_caster_joint: origin xyz=0.3 0 0.05 rpy=0 0 0 -> xyz=0.3 0 0.095 rpy=0 0 0
- joint left_wheel_joint: origin xyz=0.0 0.3 0.05 rpy=0 0 0 -> xyz=0.0 0.3 0.1 rpy=0 0 0
- joint rear_caster_joint: origin xyz=-0.3 0 0.05 rpy=0 0 0 -> xyz=-0.3 0 0.095 rpy=0 0 0
- joint right_wheel_joint: origin xyz=0.0 -0.3 0.05 rpy=0 0 0 -> xyz=0.0 -0.3 0.1 rpy=0 0 0

File: seer_description/urdf/seer_robot_base.urdf.xacro (robot description, xacro)
@@ -93,5 +93,5 @@
       <parent link="base_link" />
       <child link="${prefix}_lidar_link" />
-      <origin xyz="${x_offset*xy_reflect} ${y_offset*xy_reflect} 0.15" rpy="0 0 0" />
+      <origin xyz="${x_offset*xy_reflect} ${y_offset*xy_reflect} 0.2" rpy="0 0 0" />
     </joint>
   </xacro:macro>
@@ -110,9 +110,4 @@
     </inertial>
   </link>
-  <!-- <joint name="front_caster_joint" type="fixed">
-    <parent link="base_link" />
-    <child link="front_caster" />
-    <origin xyz="0.3 0 ${wheel_zoff}" rpy="0 0 0" />
-  </joint> -->
   <link name="rear_caster">
     <collision>
@@ -127,9 +122,4 @@
     </inertial>
   </link>
-  <!-- <joint name="rear_caster_joint" type="fixed">
-    <parent link="base_link" />
-    <child link="rear_caster" />
-    <origin xyz="-0.3 0 ${wheel_zoff}" rpy="0 0 0" />
-  </joint> -->
   <joint name="front_caster_joint" type="fixed">
     <parent link="base_link" />
@@ -173,7 +163,7 @@
       <wheel_radius>${wheel_radius}</wheel_radius>
       <max_linear_acceleration>1.0</max_linear_acceleration>
-      <max_angular_acceleration>2.0</max_angular_acceleration>
+      <max_angular_acceleration>1.0</max_angular_acceleration>
       <max_linear_velocity>1.5</max_linear_velocity>
-      <max_angular_velocity>2.0</max_angular_velocity>
+      <max_angular_velocity>0.5</max_angular_velocity>
       <topic>cmd_vel</topic>
       <odom_topic>odom</odom_topic>
@@ -189,3 +179,68 @@
     </plugin>
   </gazebo>
+  <gazebo reference="front_lidar_link">
+    <sensor name="front_lidar_sensor" type="gpu_lidar">
+      <topic>/lidar_front</topic>
+      <gz_frame_id>front_lidar_link</gz_frame_id>
+      <update_rate>10</update_rate>
+      <ray>
+        <scan>
+          <horizontal>
+            <samples>360</samples>
+            <resolution>1</resolution>
+            <min_angle>-3.14159</min_angle>
+            <max_angle>3.14159</max_angle>
+          </horizontal>
+          <vertical>
+            <samples>16</samples>
+            <resolution>1</resolution>
+            <min_angle>-0.2618</min_angle>
+            <max_angle>0.2618</max_angle>
+          </vertical>
+        </scan>
+        <range>
+          <min>0.2</min>
+          <max>30.0</max>
+          <resolution>0.01</resolution>
+        </range>
+      </ray>
+      <always_on>1</always_on>
+      <visualize>true</visualize>
+    </sensor>
+  </gazebo>
+  <gazebo reference="back_lidar_link">
+    <sensor name="back_lidar_sensor" type="gpu_lidar">
+      <topic>/lidar_back</topic>
+      <gz_frame_id>back_lidar_link</gz_frame_id>
+      <update_rate>10</update_rate>
+      <ray>
+        <scan>
+          <horizontal>
+            <samples>360</samples>
+            <resolution>1</resolution>
+            <min_angle>-3.14159</min_angle>
+            <max_angle>3.14159</max_angle>
+          </horizontal>
+          <vertical>
+            <samples>16</samples>
+            <resolution>1</resolution>
+            <min_angle>-0.2618</min_angle>
+            <max_angle>0.2618</max_angle>
+          </vertical>
+        </scan>
+        <range>
+          <min>0.2</min>
+          <max>30.0</max>
+          <resolution>0.01</resolution>
+        </range>
+      </ray>
+      <always_on>1</always_on>
+      <visualize>true</visualize>
+    </sensor>
+  </gazebo>
+<gazebo>
+    <plugin filename="gz-sim-sensors-system" name="gz::sim::systems::Sensors">
+      <render_engine>ogre2</render_engine>
+    </plugin>
+  </gazebo>
 </robot>

Commit message: configing Lidar in USD

File: seer_description/urdf/seer_robot_base.urdf (robot description, URDF)
Before this commit: robot seer_amb, 8 links, 7 joints
Joints:
- joint back_lidar_joint: origin xyz=-0.38 -0.25 0.15 rpy=0 0 0 -> xyz=-0.38 -0.25 0.2 rpy=0 0 0
- joint front_lidar_joint: origin xyz=0.38 0.25 0.15 rpy=0 0 0 -> xyz=0.38 0.25 0.2 rpy=0 0 0
