Commit message: setup usd file, need configurations

File: seer_description/urdf/composite_robot_isaac.urdf (robot description, URDF)
Before this commit: robot seer_aubo_composite, 25 links, 24 joints
Links:
- link aubo_base_link: geometry collision mesh filename=package://seer_description/meshes/aubo_i16/collision/link0.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; visual mesh filename=package://seer_description/meshes/aubo_i16/collision/link0.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
- link foreArm_Link: geometry collision mesh filename=package://seer_description/meshes/aubo_i16/collision/link3.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; visual mesh filename=package://seer_description/meshes/aubo_i16/collision/link3.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
- link shoulder_Link: geometry collision mesh filename=package://seer_description/meshes/aubo_i16/collision/link1.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; visual mesh filename=package://seer_description/meshes/aubo_i16/collision/link1.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
- link upperArm_Link: geometry collision mesh filename=package://seer_description/meshes/aubo_i16/collision/link2.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; visual mesh filename=package://seer_description/meshes/aubo_i16/collision/link2.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
- link wrist1_Link: geometry collision mesh filename=package://seer_description/meshes/aubo_i16/collision/link4.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; visual mesh filename=package://seer_description/meshes/aubo_i16/collision/link4.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
- link wrist2_Link: geometry collision mesh filename=package://seer_description/meshes/aubo_i16/collision/link5.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; visual mesh filename=package://seer_description/meshes/aubo_i16/collision/link5.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
- link wrist3_Link: geometry collision mesh filename=package://seer_description/meshes/aubo_i16/collision/link6.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; visual mesh filename=package://seer_description/meshes/aubo_i16/collision/link6.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
