Commit message: update for gazebo

File: seer_description/urdf/composite_robot.urdf.xacro (robot description, xacro)
@@ -8,3 +8,30 @@
     <origin xyz="-0.3 0.0 0.6" rpy="0 0 ${pi}" />
   </joint>
+  <ros2_control name="GazeboSimSystem" type="system">
+    <hardware>
+      <plugin>gz_ros2_control/GazeboSimSystem</plugin>
+    </hardware>
+    <xacro:macro name="aubo_joint_interface" params="joint_name">
+      <joint name="${joint_name}">
+        <command_interface name="position">
+          <param name="min">-6.28</param>
+          <param name="max">6.28</param>
+        </command_interface>
+        <state_interface name="position" />
+        <state_interface name="velocity" />
+        <state_interface name="effort" />
+      </joint>
+    </xacro:macro>
+    <xacro:aubo_joint_interface joint_name="shoulder_joint" />
+    <xacro:aubo_joint_interface joint_name="upperArm_joint" />
+    <xacro:aubo_joint_interface joint_name="foreArm_joint" />
+    <xacro:aubo_joint_interface joint_name="wrist1_joint" />
+    <xacro:aubo_joint_interface joint_name="wrist2_joint" />
+    <xacro:aubo_joint_interface joint_name="wrist3_joint" />
+  </ros2_control>
+  <gazebo>
+    <plugin filename="gz_ros2_control-system" name="gz_ros2_control::GazeboSimROS2ControlPlugin">
+      <parameters>$(find seer_description)/config/aubo_controllers.yaml</parameters>
+    </plugin>
+  </gazebo>
 </robot>

Commit message: update for camera(not tested yet)

File: seer_description/urdf/composite_robot.urdf.xacro (robot description, xacro)
@@ -35,3 +35,9 @@
     </plugin>
   </gazebo>
+  <xacro:include filename="$(find orbbec_description)/urdf/gemini335L_336L.urdf.xacro" />
+  <joint name="camera_joint" type="fixed">
+    <parent link="wrist3_Link" />
+    <child link="camera_link" />
+    <origin xyz="0.03 0.03 0.02" rpy="0 0 0" />
+  </joint>
 </robot>

Commit message: update

File: seer_description/urdf/composite_robot.urdf.xacro (robot description, xacro)
@@ -35,9 +35,9 @@
     </plugin>
   </gazebo>
-  <xacro:include filename="$(find orbbec_description)/urdf/gemini335L_336L.urdf.xacro" />
+  <xacro:include filename="$(find seer_description)/urdf/gemini335L_336L.urdf.xacro" />
   <joint name="camera_joint" type="fixed">
     <parent link="wrist3_Link" />
     <child link="camera_link" />
-    <origin xyz="0.03 0.03 0.02" rpy="0 0 0" />
+    <origin xyz="0.00 0.08 0.00" rpy="${pi/2} -${pi/2} ${pi}" />
   </joint>
 </robot>

File: seer_description/urdf/seer_robot_base.urdf.xacro (robot description, xacro)
@@ -25,12 +25,13 @@
     </visual>
     <collision>
-      <origin xyz="0 0 0.2" rpy="0 0 0" />
-      <geometry>
-        <box size="0.8 0.5 0.3" />
+      <origin xyz="0 0 0.35" rpy="0 0 0" />
+      <geometry>
+        <box size="1.00 0.70 0.50" />
       </geometry>
     </collision>
     <inertial>
       <origin xyz="0 0 0.15" rpy="0 0 0" />
-      <mass value="${base_mass}" /> <inertia ixx="3.11" ixy="0.0" ixz="0.0" iyy="6.68" iyz="0.0" izz="8.15" />
+      <mass value="${base_mass}" />
+      <inertia ixx="3.11" ixy="0.0" ixz="0.0" iyy="6.68" iyz="0.0" izz="8.15" />
     </inertial>
   </link>
@@ -81,5 +82,5 @@
         <origin xyz="0 0 0" rpy="0 0 0" />
         <geometry>
-          <cylinder radius="0.05" length="0.08"  />
+          <cylinder radius="0.05" length="0.08" />
         </geometry>
       </collision>
@@ -239,5 +240,5 @@
     </sensor>
   </gazebo>
-<gazebo>
+  <gazebo>
     <plugin filename="gz-sim-sensors-system" name="gz::sim::systems::Sensors">
       <render_engine>ogre2</render_engine>

Commit message: adding gripper

File: seer_description/urdf/composite_robot.urdf.xacro (robot description, xacro)
@@ -3,4 +3,5 @@
   <xacro:include filename="$(find seer_description)/urdf/seer_robot_base.urdf.xacro" />
   <xacro:include filename="$(find seer_description)/urdf/aubo_i16.urdf" />
+  <xacro:include filename="$(find seer_description)/urdf/gripper_stick.urdf.xacro" />
   <joint name="arm_mount_joint" type="fixed">
     <parent link="base_link" />
@@ -39,5 +40,8 @@
     <parent link="wrist3_Link" />
     <child link="camera_link" />
-    <origin xyz="0.00 0.08 0.00" rpy="${pi/2} -${pi/2} ${pi}" />
+    <origin xyz="0.00 0.1 0.00" rpy="${pi/2} -${pi/2} ${pi}" />
   </joint>
+  <xacro:my_custom_gripper parent="wrist3_Link">
+    <origin xyz="0 0 0" rpy="0 0 0" />
+  </xacro:my_custom_gripper>
 </robot>
