Commit message: Add mono end-effector camera attach to gripper motor

File: seer_description/urdf/composite_robot_stick.urdf.xacro (robot description, xacro)
@@ -39,11 +39,12 @@
   </gazebo>
   <xacro:include filename="$(find seer_description)/urdf/gemini33X_simple.urdf.xacro" />
+  <xacro:my_custom_gripper parent="wrist3_Link">
+    <origin xyz="0 0 0" rpy="0 0 0" />
+  </xacro:my_custom_gripper>
+  <!-- 末端夹爪后端安装：挂在 gripper_motor_link 上，避免停在 wrist3 中段。 -->
   <joint name="camera_joint" type="fixed">
-    <parent link="wrist3_Link" />
+    <parent link="gripper_motor_link" />
     <child link="camera_link" />
     <origin xyz="0.00 0.1 0.00" rpy="${pi/2} -${pi/2} ${pi}" />
   </joint>
-  <xacro:my_custom_gripper parent="wrist3_Link">
-    <origin xyz="0 0 0" rpy="0 0 0" />
-  </xacro:my_custom_gripper>
 </robot>

File: seer_description/urdf/composite_robot_stick_mono.urdf (robot description, URDF)
Before this commit: robot seer_aubo_composite, 21 links, 20 joints
Joints:
- joint camera_joint: parent wrist3_Link -> gripper_motor_link

File: seer_description/urdf/composite_robot_stick_mono.urdf.xacro (robot description, xacro)
@@ -39,11 +39,12 @@
   </gazebo>
   <xacro:include filename="$(find seer_description)/urdf/mv_ch100_60um_12mm.urdf.xacro" />
+  <xacro:my_custom_gripper parent="wrist3_Link">
+    <origin xyz="0 0 0" rpy="0 0 0" />
+  </xacro:my_custom_gripper>
+  <!-- 末端夹爪后端安装：挂在 gripper_motor_link 上，避免停在 wrist3 中段。 -->
   <joint name="camera_joint" type="fixed">
-    <parent link="wrist3_Link" />
+    <parent link="gripper_motor_link" />
     <child link="camera_link" />
     <origin xyz="0.00 0.1 0.00" rpy="0 0 ${pi}" />
   </joint>
-  <xacro:my_custom_gripper parent="wrist3_Link">
-    <origin xyz="0 0 0" rpy="0 0 0" />
-  </xacro:my_custom_gripper>
 </robot>

Commit message: Restore validated wrist camera mount across model formats

File: seer_description/urdf/composite_robot_stick.urdf.xacro (robot description, xacro)
@@ -42,7 +42,7 @@
     <origin xyz="0 0 0" rpy="0 0 0" />
   </xacro:my_custom_gripper>
-  <!-- 末端夹爪后端安装：挂在 gripper_motor_link 上，避免停在 wrist3 中段。 -->
+  <!-- 相机安装与已验证的 Ubuntu 运行模型一致，固定在腕部坐标系。 -->
   <joint name="camera_joint" type="fixed">
-    <parent link="gripper_motor_link" />
+    <parent link="wrist3_Link" />
     <child link="camera_link" />
     <origin xyz="0.00 0.1 0.00" rpy="${pi/2} -${pi/2} ${pi}" />

File: seer_description/urdf/composite_robot_stick_mono.urdf (robot description, URDF)
Before this commit: robot seer_aubo_composite, 21 links, 20 joints
Joints:
- joint camera_joint: parent gripper_motor_link -> wrist3_Link

File: seer_description/urdf/composite_robot_stick_mono.urdf.xacro (robot description, xacro)
@@ -42,7 +42,7 @@
     <origin xyz="0 0 0" rpy="0 0 0" />
   </xacro:my_custom_gripper>
-  <!-- 末端夹爪后端安装：挂在 gripper_motor_link 上，避免停在 wrist3 中段。 -->
+  <!-- 相机安装与已验证的 Ubuntu 运行模型一致，固定在腕部坐标系。 -->
   <joint name="camera_joint" type="fixed">
-    <parent link="gripper_motor_link" />
+    <parent link="wrist3_Link" />
     <child link="camera_link" />
     <origin xyz="0.00 0.1 0.00" rpy="0 0 ${pi}" />
