Commit message: reset urdf

File: seer_description/urdf/composite_robot.urdf (robot description, URDF)
Before this commit: robot seer_aubo_composite, 29 links, 28 joints
Links:
- removed link gripper1_link
- removed link gripper2_link
- removed link gripper_adapter_link
- removed link gripper_motor_link
Joints:
- removed joint adapter_mount_joint
- removed joint gripper1_joint
- removed joint gripper2_joint
- removed joint motor_mount_joint
