Commit message: update but not tested

File: seer_description/urdf/aubo_i16H_simple.urdf.xacro (robot description, xacro)
@@ -7,6 +7,6 @@
     for faster physics computation.
   -->
-  <dh_type type="modified"/>
-  <safety_para singularity_consistent="0.02 0.01 10 0.2 0.045 10"/>
+  <dh_type type="modified" />
+  <safety_para singularity_consistent="0.02 0.01 10 0.2 0.045 10" />
   <!--
     Collision primitives guide for i16H:
@@ -23,10 +23,11 @@
       <origin xyz="0.000136 0.001601 0.018986" rpy="0 0 0" />
       <mass value="2.592000" />
-      <inertia ixx="0.008524" ixy="-0.000001" ixz="-0.000005" iyy="0.007934" iyz="-0.000081" izz="0.015304" />
-    </inertial>
-    <visual>
-      <origin xyz="0 0 0" rpy="0 0 0" />
-      <geometry>
-        <mesh filename="package://aubo_description/meshes/aubo_i16H/visual/link0.DAE" />
+      <inertia ixx="0.008524" ixy="-0.000001" ixz="-0.000005" iyy="0.007934" iyz="-0.000081"
+        izz="0.015304" />
+    </inertial>
+    <visual>
+      <origin xyz="0 0 0" rpy="0 0 0" />
+      <geometry>
+        <mesh filename="package://seer_description/meshes/aubo_i16H/visual/link0.DAE" />
       </geometry>
       <material name="">
@@ -46,10 +47,11 @@
       <origin xyz="-0.000004 0.005112 -0.026275" rpy="0 0 0" />
       <mass value="10.180139" />
-      <inertia ixx="0.043326" ixy="0.000003" ixz="0.000003" iyy="0.042233" iyz="-0.001767" izz="0.029902" />
-    </inertial>
-    <visual>
-      <origin xyz="0 0 0" rpy="0 0 0" />
-      <geometry>
-        <mesh filename="package://aubo_description/meshes/aubo_i16H/visual/link1.DAE" />
+      <inertia ixx="0.043326" ixy="0.000003" ixz="0.000003" iyy="0.042233" iyz="-0.001767"
+        izz="0.029902" />
+    </inertial>
+    <visual>
+      <origin xyz="0 0 0" rpy="0 0 0" />
+      <geometry>
+        <mesh filename="package://seer_description/meshes/aubo_i16H/visual/link1.DAE" />
       </geometry>
       <material name="">
@@ -70,5 +72,6 @@
     <child link="shoulder_Link" />
     <axis xyz="0 0 1" />
-    <limit lower="-6.283185307179586" upper="6.283185307179586" effort="267" start_stop="411" velocity="3.106686068549906" />
+    <limit lower="-6.283185307179586" upper="6.283185307179586" effort="267" start_stop="411"
+      velocity="3.106686068549906" />
   </joint>
   <link name="upperArm_Link">
@@ -76,10 +79,11 @@
       <origin xyz="0.170602 0.000000 -0.013024" rpy="0 0 0" />
       <mass value="17.664060" />
-      <inertia ixx="0.063521" ixy="0.000020" ixz="-0.024888" iyy="0.847528" iyz="0.000005" izz="0.828847" />
-    </inertial>
-    <visual>
-      <origin xyz="0 0 0" rpy="0 0 0" />
-      <geometry>
-        <mesh filename="package://aubo_description/meshes/aubo_i16H/visual/link2.DAE" />
+      <inertia ixx="0.063521" ixy="0.000020" ixz="-0.024888" iyy="0.847528" iyz="0.000005"
+        izz="0.828847" />
+    </inertial>
+    <visual>
+      <origin xyz="0 0 0" rpy="0 0 0" />
+      <geometry>
+        <mesh filename="package://seer_description/meshes/aubo_i16H/visual/link2.DAE" />
       </geometry>
       <material name="">
@@ -96,9 +100,11 @@
   </link>
   <joint name="upperArm_joint" type="revolute">
-    <origin xyz="0 0.191 0" rpy="-1.5707963267948966192313216916398 -1.5707963267948966192313216916398 0" />
+    <origin xyz="0 0.191 0"
+      rpy="-1.5707963267948966192313216916398 -1.5707963267948966192313216916398 0" />
     <parent link="shoulder_Link" />
     <child link="upperArm_Link" />
     <axis xyz="0 0 1" />
-    <limit lower="-6.283185307179586" upper="6.283185307179586" effort="267" start_stop="411" velocity="3.106686068549906" />
+    <limit lower="-6.283185307179586" upper="6.283185307179586" effort="267" start_stop="411"
+      velocity="3.106686068549906" />
   </joint>
   <link name="foreArm_Link">
@@ -106,10 +112,11 @@
       <origin xyz="0.269208 -0.000022 0.106467" rpy="0 0 0" />
       <mass value="3.926354" />
-      <inertia ixx="0.006007" ixy="0.000009" ixz="0.001991" iyy="0.083780" iyz="0.000005" izz="0.082433" />
-    </inertial>
-    <visual>
-      <origin xyz="0 0 0" rpy="0 0 0" />
-      <geometry>
-        <mesh filename="package://aubo_description/meshes/aubo_i16H/visual/link3.DAE" />
+      <inertia ixx="0.006007" ixy="0.000009" ixz="0.001991" iyy="0.083780" iyz="0.000005"
+        izz="0.082433" />
+    </inertial>
+    <visual>
+      <origin xyz="0 0 0" rpy="0 0 0" />
+      <geometry>
+        <mesh filename="package://seer_description/meshes/aubo_i16H/visual/link3.DAE" />
       </geometry>
       <material name="">
@@ -130,5 +137,6 @@
     <child link="foreArm_Link" />
     <axis xyz="0 0 1" />
-    <limit lower="-6.283185307179586" upper="6.283185307179586" effort="133" start_stop="207" velocity="4.660029102824860" />
+    <limit lower="-6.283185307179586" upper="6.283185307179586" effort="133" start_stop="207"
+      velocity="4.660029102824860" />
   </joint>
   <link name="wrist1_Link">
@@ -136,10 +144,11 @@
       <origin xyz="0.000036 0.015610 -0.001526" rpy="0 0 0" />
       <mass value="2.370741" />
-      <inertia ixx="0.003672" ixy="0.000006" ixz="-0.000001" iyy="0.002190" iyz="-0.000080" izz="0.003621" />
-    </inertial>
-    <visual>
-      <origin xyz="0 0 0" rpy="0 0 0" />
-      <geometry>
-        <mesh filename="package://aubo_description/meshes/aubo_i16H/visual/link4.DAE" />
+      <inertia ixx="0.003672" ixy="0.000006" ixz="-0.000001" iyy="0.002190" iyz="-0.000080"
+        izz="0.003621" />
+    </inertial>
+    <visual>
+      <origin xyz="0 0 0" rpy="0 0 0" />
+      <geometry>
+        <mesh filename="package://seer_description/meshes/aubo_i16H/visual/link4.DAE" />
       </geometry>
       <material name="">
@@ -156,9 +165,11 @@
   </link>
   <joint name="wrist1_joint" type="revolute">
-    <origin xyz="0.370 0 0" rpy="3.1415926535897932384626433832795 -1.4294E-15 1.5707963267948966192313216916398" />
+    <origin xyz="0.370 0 0"
+      rpy="3.1415926535897932384626433832795 -1.4294E-15 1.5707963267948966192313216916398" />
     <parent link="foreArm_Link" />
     <child link="wrist1_Link" />
     <axis xyz="0 0 1" />
-    <limit lower="-6.283185307179586" upper="6.283185307179586" effort="49" start_stop="66" velocity="4.136430327226561" />
+    <limit lower="-6.283185307179586" upper="6.283185307179586" effort="49" start_stop="66"
+      velocity="4.136430327226561" />
   </joint>
   <link name="wrist2_Link">
@@ -166,10 +177,11 @@
       <origin xyz="-0.000036 -0.015610 -0.001526" rpy="0 0 0" />
       <mass value="2.370741" />
-      <inertia ixx="0.003672" ixy="0.000006" ixz="0.000001" iyy="0.002190" iyz="0.000080" izz="0.003621" />
-    </inertial>
-    <visual>
-      <origin xyz="0 0 0" rpy="0 0 0" />
-      <geometry>
-        <mesh filename="package://aubo_description/meshes/aubo_i16H/visual/link5.DAE" />
+      <inertia ixx="0.003672" ixy="0.000006" ixz="0.000001" iyy="0.002190" iyz="0.000080"
+        izz="0.003621" />
+    </inertial>
+    <visual>
+      <origin xyz="0 0 0" rpy="0 0 0" />
+      <geometry>
+        <mesh filename="package://seer_description/meshes/aubo_i16H/visual/link5.DAE" />
       </geometry>
       <material name="">
@@ -190,5 +202,6 @@
     <child link="wrist2_Link" />
     <axis xyz="0 0 1" />
-    <limit lower="-6.283185307179586" upper="6.283185307179586" effort="49" start_stop="66" velocity="4.136430327226561" />
+    <limit lower="-6.283185307179586" upper="6.283185307179586" effort="49" start_stop="66"
+      velocity="4.136430327226561" />
   </joint>
   <link name="wrist3_Link">
@@ -196,10 +209,11 @@
       <origin xyz="0.000508 0.000344 -0.017049" rpy="0 0 0" />
       <mass value="0.259654" />
-      <inertia ixx="0.000162" ixy="-0.000000" ixz="-0.000000" iyy="0.000160" iyz="0.000001" izz="0.000273" />
-    </inertial>
-    <visual>
-      <origin xyz="0 0 0" rpy="0 0 0" />
-      <geometry>
-        <mesh filename="package://aubo_description/meshes/aubo_i16H/visual/link6.DAE" />
+      <inertia ixx="0.000162" ixy="-0.000000" ixz="-0.000000" iyy="0.000160" iyz="0.000001"
+        izz="0.000273" />
+    </inertial>
+    <visual>
+      <origin xyz="0 0 0" rpy="0 0 0" />
+      <geometry>
+        <mesh filename="package://seer_description/meshes/aubo_i16H/visual/link6.DAE" />
       </geometry>
       <material name="">
@@ -220,10 +234,11 @@
     <child link="wrist3_Link" />
     <axis xyz="0 0 1" />
-    <limit lower="-6.283185307179586" upper="6.283185307179586" effort="49" start_stop="66" velocity="4.136430327226561" />
+    <limit lower="-6.283185307179586" upper="6.283185307179586" effort="49" start_stop="66"
+      velocity="4.136430327226561" />
   </joint>
   <link name="world" />
   <joint name="world_joint" type="fixed">
     <parent link="world" />
-    <child link = "base_link" />
+    <child link="base_link" />
     <origin xyz="0.0 0.0 0.0" rpy="0.0 0.0 0.0" />
   </joint>
