Commit message: set up simplified model for less computational cost

File: seer_description/urdf/aubo_i16H_simple.urdf (robot description, URDF)
Before this commit: robot aubo_i16H_simple, 8 links, 7 joints
Links:
- removed link base_link
- removed link world
- added link aubo_base_link, mass 2.592000; collision cylinder length=0.163 radius=0.06; visual mesh filename=package://seer_description/meshes/aubo_i16H/visual/link0.DAE
- link foreArm_Link: geometry collision cylinder length=0.370 radius=0.035; visual mesh filename=package://seer_description/meshes/aubo_i16H/visual/link3.DAE
- link shoulder_Link: geometry collision sphere radius=0.08; visual mesh filename=package://seer_description/meshes/aubo_i16H/visual/link1.DAE
- link upperArm_Link: geometry collision cylinder length=0.55 radius=0.045; visual mesh filename=package://seer_description/meshes/aubo_i16H/visual/link2.DAE
- link wrist1_Link: geometry collision sphere radius=0.045; visual mesh filename=package://seer_description/meshes/aubo_i16H/visual/link4.DAE
- link wrist2_Link: geometry collision sphere radius=0.045; visual mesh filename=package://seer_description/meshes/aubo_i16H/visual/link5.DAE
- link wrist3_Link: geometry collision sphere radius=0.035; visual mesh filename=package://seer_description/meshes/aubo_i16H/visual/link6.DAE
Joints:
- removed joint world_joint
- joint shoulder_joint: parent base_link -> aubo_base_link

File: seer_description/urdf/aubo_i16H_simple.urdf.xacro (robot description, xacro)
@@ -19,5 +19,5 @@
     - link6 (wrist3/TCP): sphere r=0.035
   -->
-  <link name="base_link">
+  <link name="aubo_base_link">
     <inertial>
       <origin xyz="0.000136 0.001601 0.018986" rpy="0 0 0" />
@@ -69,5 +69,5 @@
   <joint name="shoulder_joint" type="revolute">
     <origin xyz="0 0 0.163" rpy="-8.7138E-17 -4.3534E-32 3.1415926535897932384626433832795" />
-    <parent link="base_link" />
+    <parent link="aubo_base_link" />
     <child link="shoulder_Link" />
     <axis xyz="0 0 1" />
@@ -93,7 +93,7 @@
     <!-- Upper arm: long cylinder along the link -->
     <collision>
-      <origin xyz="0.24 0 0" rpy="0 0 0" />
-      <geometry>
-        <cylinder radius="0.045" length="0.480" />
+      <origin xyz="0.26 0 0" rpy="0 1.5707963267948966192313216916398 0" />
+      <geometry>
+        <cylinder radius="0.045" length="0.55" />
       </geometry>
     </collision>
@@ -124,7 +124,7 @@
       </material>
     </visual>
-    <!-- Forearm: cylinder -->
-    <collision>
-      <origin xyz="0.185 0 0" rpy="0 0 0" />
+    <!-- Forearm: cylinder 0.185-->
+    <collision>
+      <origin xyz="0.19 0. 0.12" rpy="0 1.5707963267948966192313216916398 0" />
       <geometry>
         <cylinder radius="0.035" length="0.370" />
@@ -237,9 +237,12 @@
       velocity="4.136430327226561" />
   </joint>
-  <link name="world" />
+  <!-- using world if you only use this urdf alone, but when included in
+  composite_robot_stick.xacro, the world link and joint are defined there, so we comment them out
+  here to avoid duplication. -->
+  <!-- <link name="world" />
   <joint name="world_joint" type="fixed">
     <parent link="world" />
     <child link="base_link" />
     <origin xyz="0.0 0.0 0.0" rpy="0.0 0.0 0.0" />
-  </joint>
+  </joint> -->
 </robot>

File: seer_description/urdf/composite_robot_stick.urdf (robot description, URDF)
Before this commit: robot seer_aubo_composite, 29 links, 28 joints
Links:
- link aubo_base_link: mass 2.592 -> 2.592000; geometry collision cylinder length=0.163 radius=0.06; visual mesh filename=package://seer_description/meshes/aubo_i16H/visual/link0.DAE
- link camera_IMU_frame: geometry collision box size=0.01 0.01 0.005; visual mesh filename=package://seer_description/meshes/gemini335L_336L/camera_IM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
- link camera_color_frame: geometry collision box size=0.04 0.03 0.015; visual mesh filename=package://seer_description/meshes/gemini335L_336L/camera_co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
- link camera_color_optical_frame: geometry collision box size=0.008 0.008 0.008; visual mesh filename=package://seer_description/meshes/gemini335L_336L/camera_co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
- link camera_color_screw_frame: geometry collision box size=0.04 0.015 0.005; visual mesh filename=package://seer_description/meshes/gemini335L_336L/camera_co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
- link camera_depth_frame: geometry collision box size=0.065 0.05 0.02; visual mesh filename=package://seer_description/meshes/gemini335L_336L/camera_de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
- link camera_left_ir_frame: geometry collision box size=0.04 0.03 0.015; visual mesh filename=package://seer_description/meshes/gemini335L_336L/camera_in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
- link camera_left_ir_optical_frame: geometry collision box size=0.008 0.008 0.008; visual mesh filename=package://seer_description/meshes/gemini335L_336L/camera_in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
- link camera_link: geometry collision box size=0.07 0.05 0.035; visual mesh filename=package://seer_description/meshes/gemini335L_336L/base_link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
- link camera_right_ir_frame: geometry collision box size=0.04 0.03 0.015; visual mesh filename=package://seer_description/meshes/gemini335L_336L/camera_in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
- link camera_right_ir_optical_frame: geometry collision box size=0.008 0.008 0.008; visual mesh filename=package://seer_description/meshes/gemini335L_336L/camera_in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
- link foreArm_Link: geometry collision cylinder length=0.370 radius=0.035; visual mesh filename=package://seer_description/meshes/aubo_i16H/visual/link3.DAE
- link gripper_adapter_link: geometry collision box size=0.1 0.1 0.05; visual mesh filename=package://seer_description/meshes/adapter.stl scale=1 1 1
- link gripper_motor_link: geometry collision cylinder length=0.14 radius=0.025; visual mesh filename=package://seer_description/meshes/motor.stl scale=1 1 1
- link shoulder_Link: geometry collision sphere radius=0.08; visual mesh filename=package://seer_description/meshes/aubo_i16H/visual/link1.DAE
- link upperArm_Link: mass 17.66406 -> 17.664060; geometry collision cylinder length=0.55 radius=0.045; visual mesh filename=package://seer_description/meshes/aubo_i16H/visual/link2.DAE
- link wrist1_Link: geometry collision sphere radius=0.045; visual mesh filename=package://seer_description/meshes/aubo_i16H/visual/link4.DAE
- link wrist2_Link: geometry collision sphere radius=0.045; visual mesh filename=package://seer_description/meshes/aubo_i16H/visual/link5.DAE
- link wrist3_Link: geometry collision sphere radius=0.035; visual mesh filename=package://seer_description/meshes/aubo_i16H/visual/link6.DAE
Joints:
- joint foreArm_joint: limit lower=-6.283185307179586476925286766559 upper=6.283185307179586476925286766559 effort=133 velocity=4.6600 -> lower=-6.283185307179586 upper=6.283185307179586 effort=133 velocity=4.660029102824860; origin xyz=0.480 0 0 rpy=-3.1415926535897932384626433832795 0 0 -> xyz=0.480 0 0 rpy=-3.1415926535897932384626433832795 -4.5954E-17 -8.4328E-17
- joint shoulder_joint: limit lower=-6.283185307179586476925286766559 upper=6.283185307179586476925286766559 effort=267 velocity=3.1416 -> lower=-6.283185307179586 upper=6.283185307179586 effort=267 velocity=3.106686068549906; origin xyz=0 0 0.163 rpy=0 0 3.1415926535897932384626433832795 -> xyz=0 0 0.163 rpy=-8.7138E-17 -4.3534E-32 3.1415926535897932384626433832795
- joint upperArm_joint: limit lower=-6.283185307179586476925286766559 upper=6.283185307179586476925286766559 effort=267 velocity=3.1416 -> lower=-6.283185307179586 upper=6.283185307179586 effort=267 velocity=3.106686068549906
- joint wrist1_joint: limit lower=-6.283185307179586476925286766559 upper=6.283185307179586476925286766559 effort=49 velocity=3.1416 -> lower=-6.283185307179586 upper=6.283185307179586 effort=49 velocity=4.136430327226561; origin xyz=0.370 0 0 rpy=3.1415926535897932384626433832795 0 1.5707963267948966192313216916398 -> xyz=0.370 0 0 rpy=3.1415926535897932384626433832795 -1.4294E-15 1.5707963267948966192313216916398
- joint wrist2_joint: limit lower=-6.283185307179586476925286766559 upper=6.283185307179586476925286766559 effort=49 velocity=3.1416 -> lower=-6.283185307179586 upper=6.283185307179586 effort=49 velocity=4.136430327226561; origin xyz=0 0.1175 0 rpy=-1.5707963267948966192313216916398 0 0 -> xyz=0 0.1175 0 rpy=-1.5707963267948966192313216916398 -7.0777E-16 -7.4101E-16
- joint wrist3_joint: limit lower=-6.283185307179586476925286766559 upper=6.283185307179586476925286766559 effort=49 velocity=3.1416 -> lower=-6.283185307179586 upper=6.283185307179586 effort=49 velocity=4.136430327226561; origin xyz=0 -0.1035 0 rpy=1.5707963267948966192313216916398 0 0 -> xyz=0 -0.1035 0 rpy=1.5707963267948966192313216916398 0 6.7283E-16

File: seer_description/urdf/composite_robot_stick.urdf.xacro (robot description, xacro)
@@ -2,6 +2,6 @@
 <robot name="seer_aubo_composite" xmlns:xacro="http://ros.org/wiki/xacro">
   <xacro:include filename="$(find seer_description)/urdf/seer_robot_base.urdf.xacro" />
-  <xacro:include filename="$(find seer_description)/urdf/aubo_i16.urdf" />
-  <xacro:include filename="$(find seer_description)/urdf/gripper_stick.urdf.xacro" />
+  <xacro:include filename="$(find seer_description)/urdf/aubo_i16H_simple.urdf" />
+  <xacro:include filename="$(find seer_description)/urdf/gripper_stick_simple.urdf.xacro" />
   <joint name="arm_mount_joint" type="fixed">
     <parent link="base_link" />
@@ -38,5 +38,5 @@
     </plugin>
   </gazebo>
-  <xacro:include filename="$(find seer_description)/urdf/gemini335L_336L.urdf.xacro" />
+  <xacro:include filename="$(find seer_description)/urdf/gemini33X_simple.urdf.xacro" />
   <joint name="camera_joint" type="fixed">
     <parent link="wrist3_Link" />
