Commit message: fix: enforce i16H J3 limits of plus or minus 161 degrees across simulation

File: seer_description/urdf/aubo_i16H.urdf (robot description, URDF)
Before this commit: robot aubo_i16H, 8 links, 7 joints
Joints:
- joint foreArm_joint: limit lower=-6.283185307179586 upper=6.283185307179586 effort=133 velocity=4.660029102824860 -> lower=-2.8099800957108707 upper=2.8099800957108707 effort=133 velocity=4.660029102824860

File: seer_description/urdf/aubo_i16H.urdf.xacro (robot description, xacro)
@@ -111,5 +111,5 @@
     <child link="foreArm_Link" />
     <axis xyz="0 0 1" />
-    <limit lower="-6.283185307179586" upper="6.283185307179586" effort="133" start_stop="207" velocity="4.660029102824860" />
+    <limit lower="-2.8099800957108707" upper="2.8099800957108707" effort="133" start_stop="207" velocity="4.660029102824860" />
   </joint>
   <link name="wrist1_Link">

File: seer_description/urdf/aubo_i16H_simple.urdf (robot description, URDF)
Before this commit: robot aubo_i16H_simple, 7 links, 6 joints
Joints:
- joint foreArm_joint: limit lower=-6.283185307179586 upper=6.283185307179586 effort=133 velocity=4.660029102824860 -> lower=-2.8099800957108707 upper=2.8099800957108707 effort=133 velocity=4.660029102824860

File: seer_description/urdf/aubo_i16H_simple.urdf.xacro (robot description, xacro)
@@ -137,5 +137,5 @@
     <child link="foreArm_Link" />
     <axis xyz="0 0 1" />
-    <limit lower="-6.283185307179586" upper="6.283185307179586" effort="133" start_stop="207"
+    <limit lower="-2.8099800957108707" upper="2.8099800957108707" effort="133" start_stop="207"
       velocity="4.660029102824860" />
   </joint>

File: seer_description/urdf/composite_robot_stick.urdf (robot description, URDF)
Before this commit: robot seer_aubo_composite, 29 links, 28 joints
Joints:
- joint foreArm_joint: limit lower=-6.283185307179586 upper=6.283185307179586 effort=133 velocity=4.660029102824860 -> lower=-2.8099800957108707 upper=2.8099800957108707 effort=133 velocity=4.660029102824860

File: seer_description/urdf/composite_robot_stick_mono.urdf (robot description, URDF)
Before this commit: robot seer_aubo_composite, 21 links, 20 joints
Joints:
- joint foreArm_joint: limit lower=-6.283185307179586 upper=6.283185307179586 effort=133 velocity=4.660029102824860 -> lower=-2.8099800957108707 upper=2.8099800957108707 effort=133 velocity=4.660029102824860
