Commit message: Align finger gripper physics with Blender origins

File: seer_description/urdf/composite_robot_finger_mono.urdf (robot description, URDF)
Before this commit: robot seer_aubo_composite, 21 links, 20 joints
Links:
- link gripper1_link: geometry collision box size=0.049 0.15 0.047786; visual mesh filename=package://seer_description/meshes/finger_centered.stl scale=1 1 1
- link gripper2_link: geometry collision box size=0.049 0.15 0.047786; visual mesh filename=package://seer_description/meshes/finger_centered.stl scale=1 1 1
- link gripper_motor_link: geometry collision box size=0.1985 0.063 0.137; visual mesh filename=package://seer_description/meshes/motor_new.stl scale=1 1 1
Joints:
- joint gripper1_joint: limit lower=0 upper=0.04 effort=50 velocity=0.1 -> lower=0 upper=0.0285 effort=50 velocity=0.1; origin xyz=-0.1 0 0.115 rpy=0 0 0 -> xyz=-0.0564 0 0.135 rpy=0 0 0
- joint gripper2_joint: limit lower=0 upper=0.04 effort=50 velocity=0.1 -> lower=0 upper=0.0285 effort=50 velocity=0.1; origin xyz=0.1 0 0.115 rpy=0 0 0 -> xyz=0.0564 0 0.135 rpy=0 0 0

File: seer_description/urdf/composite_robot_finger_mono.urdf.xacro (robot description, xacro)
@@ -28,6 +28,6 @@
     <xacro:aubo_joint_interface joint_name="wrist2_joint" joint_min="-6.28" joint_max="6.28"/>
     <xacro:aubo_joint_interface joint_name="wrist3_joint" joint_min="-6.28" joint_max="6.28"/>
-    <xacro:aubo_joint_interface joint_name="gripper1_joint" joint_min="0" joint_max="0.04"/>
-    <xacro:aubo_joint_interface joint_name="gripper2_joint" joint_min="0" joint_max="0.04"/>
+    <xacro:aubo_joint_interface joint_name="gripper1_joint" joint_min="0" joint_max="0.0285"/>
+    <xacro:aubo_joint_interface joint_name="gripper2_joint" joint_min="0" joint_max="0.0285"/>
   </ros2_control>
   <gazebo>

File: seer_description/urdf/gripper_finger_motor_adapter.urdf.xacro (robot description, xacro)
@@ -3,6 +3,6 @@
   <!--
     Alternative two-finger gripper made from the user-supplied millimetre STL files.
-    Joint names and 0=open / 0.04=closed semantics intentionally match the existing
-    stick gripper so the ROS 2 control, MoveIt and GUI interfaces stay unchanged.
+    Joint names intentionally match the existing stick gripper. This Blender-centred
+    geometry uses 0=open / 0.0285=closed to retain clearance between collision boxes.
   -->
   <xacro:macro name="finger_motor_adapter_gripper" params="parent *origin">
@@ -20,8 +20,8 @@
     <link name="gripper_motor_link">
       <visual>
-        <!-- Source bounds: X 0.750..199.250, Y 0.315..63.315, Z 0.630..137.630 mm. -->
-        <origin xyz="-0.1 -0.031815 -0.00063" rpy="0 0 0"/>
+        <!-- Blender-adjusted metre mesh; rotate its negative Z extent away from the wrist. -->
+        <origin xyz="0 0 0" rpy="${pi} 0 0"/>
         <geometry>
-          <mesh filename="package://seer_description/meshes/motor_adapter.STL" scale="0.001 0.001 0.001"/>
+          <mesh filename="package://seer_description/meshes/motor_new.stl" scale="1 1 1"/>
         </geometry>
         <material name="new_gripper_dark">
@@ -31,12 +31,13 @@
       <!-- Conservative primitive avoids a 42k-face planning/physics collider. -->
       <collision>
-        <origin xyz="0 0 0.0685" rpy="0 0 0"/>
+        <!-- Axis-aligned bounds after the visual's 180 degree X rotation. -->
+        <origin xyz="0.021777213 -0.000106815 0.067125965" rpy="0 0 0"/>
         <geometry><box size="0.1985 0.063 0.137"/></geometry>
       </collision>
       <inertial>
-        <!-- Temporary 1.2 kg box estimate; replace after weighing the assembly. -->
-        <origin xyz="0 0 0.0685"/>
+        <!-- Temporary 1.2 kg bounding-box estimate; replace after weighing the assembly. -->
+        <origin xyz="0.021777213 -0.000106815 0.067125965"/>
         <mass value="1.2"/>
-        <inertia ixx="0.00227" ixy="0" ixz="0" iyy="0.00588" iyz="0" izz="0.00437"/>
+        <inertia ixx="0.0022738" ixy="0" ixz="0" iyy="0.005817125" iyz="0" izz="0.004337125"/>
       </inertial>
     </link>
@@ -48,53 +49,53 @@
     <link name="gripper1_link">
       <visual>
-        <!-- Centre the 47.786 mm mesh thickness on the link Y axis. -->
-        <origin xyz="0 -0.023892963 0" rpy="0 0 0"/>
+        <!-- Blender-adjusted metre mesh; rotate its 150 mm length onto link Y. -->
+        <origin xyz="0 0 0" rpy="${-pi/2} 0 0"/>
         <geometry>
-          <mesh filename="package://seer_description/meshes/finger.STL" scale="0.001 0.001 0.001"/>
+          <mesh filename="package://seer_description/meshes/finger_centered.stl" scale="1 1 1"/>
         </geometry>
         <material name="new_gripper_finger"><color rgba="0.76 0.78 0.82 1"/></material>
       </visual>
       <collision>
-        <origin xyz="0.0245 0 0.075"/>
-        <geometry><box size="0.049 0.047786 0.15"/></geometry>
+        <origin xyz="0.003100952 0.000095278 0.024519681"/>
+        <geometry><box size="0.049 0.15 0.047786"/></geometry>
       </collision>
       <inertial>
-        <origin xyz="0.0245 0 0.075"/>
+        <origin xyz="0.003100952 0.000095278 0.024519681"/>
         <mass value="0.18"/>
-        <inertia ixx="0.00037" ixy="0" ixz="0" iyy="0.00037" iyz="0" izz="0.00007"/>
+        <inertia ixx="0.000371752" ixy="0" ixz="0" iyy="0.000070267" iyz="0" izz="0.000373515"/>
       </inertial>
     </link>
     <link name="gripper2_link">
       <visual>
-        <origin xyz="0 0.023892963 0" rpy="0 0 ${pi}"/>
+        <origin xyz="0 0 0" rpy="${-pi/2} 0 ${pi}"/>
         <geometry>
-          <mesh filename="package://seer_description/meshes/finger.STL" scale="0.001 0.001 0.001"/>
+          <mesh filename="package://seer_description/meshes/finger_centered.stl" scale="1 1 1"/>
         </geometry>
         <material name="new_gripper_finger"/>
       </visual>
       <collision>
-        <origin xyz="-0.0245 0 0.075"/>
-        <geometry><box size="0.049 0.047786 0.15"/></geometry>
+        <origin xyz="-0.003100952 -0.000095278 0.024519681"/>
+        <geometry><box size="0.049 0.15 0.047786"/></geometry>
       </collision>
       <inertial>
-        <origin xyz="-0.0245 0 0.075"/>
+        <origin xyz="-0.003100952 -0.000095278 0.024519681"/>
         <mass value="0.18"/>
-        <inertia ixx="0.00037" ixy="0" ixz="0" iyy="0.00037" iyz="0" izz="0.00007"/>
+        <inertia ixx="0.000371752" ixy="0" ixz="0" iyy="0.000070267" iyz="0" izz="0.000373515"/>
       </inertial>
     </link>
-    <!-- Meshes are 200 mm wide at q=0. Increasing q moves both fingers inward. -->
+    <!-- Blender-adjusted joint centres are 112.8 mm apart at q=0. -->
     <joint name="gripper1_joint" type="prismatic">
       <parent link="gripper_motor_link"/>
       <child link="gripper1_link"/>
-      <origin xyz="-0.1 0 0.115" rpy="0 0 0"/>
+      <origin xyz="-0.0564 0 0.135" rpy="0 0 0"/>
       <axis xyz="1 0 0"/>
-      <limit lower="0" upper="0.04" effort="50" velocity="0.1"/>
+      <limit lower="0" upper="0.0285" effort="50" velocity="0.1"/>
     </joint>
     <joint name="gripper2_joint" type="prismatic">
       <parent link="gripper_motor_link"/>
       <child link="gripper2_link"/>
-      <origin xyz="0.1 0 0.115" rpy="0 0 0"/>
+      <origin xyz="0.0564 0 0.135" rpy="0 0 0"/>
       <axis xyz="-1 0 0"/>
-      <limit lower="0" upper="0.04" effort="50" velocity="0.1"/>
+      <limit lower="0" upper="0.0285" effort="50" velocity="0.1"/>
     </joint>
   </xacro:macro>
