Commit message: update for moveit2

File: seer_aubo_moveit_config/config/seer_aubo_composite.ros2_control.xacro (robot description, xacro)
@@ -50,4 +50,18 @@
                 <state_interface name="velocity"/>
             </joint>
+            <joint name="gripper1_joint">
+                <command_interface name="position"/>
+                <state_interface name="position">
+                  <param name="initial_value">${initial_positions['gripper1_joint']}</param>
+                </state_interface>
+                <state_interface name="velocity"/>
+            </joint>
+            <joint name="gripper2_joint">
+                <command_interface name="position"/>
+                <state_interface name="position">
+                  <param name="initial_value">${initial_positions['gripper2_joint']}</param>
+                </state_interface>
+                <state_interface name="velocity"/>
+            </joint>
         </ros2_control>
     </xacro:macro>

File: seer_description/urdf/composite_robot.urdf (robot description, URDF)
Before this commit: robot seer_aubo_composite, 25 links, 24 joints
Links:
- added link gripper1_link, mass 0.3; collision mesh filename=package://seer_description/meshes/gripper_stick.stl scale=1 1 1; visual mesh filename=package://seer_description/meshes/gripper_stick.stl scale=1 1 1
- added link gripper2_link, mass 0.3; collision mesh filename=package://seer_description/meshes/gripper_stick.stl scale=1 1 1; visual mesh filename=package://seer_description/meshes/gripper_stick.stl scale=1 1 1
- added link gripper_adapter_link, mass 0.2; collision mesh filename=package://seer_description/meshes/adapter.stl scale=1 1 1; visual mesh filename=package://seer_description/meshes/adapter.stl scale=1 1 1
- added link gripper_motor_link, mass 0.5; collision mesh filename=package://seer_description/meshes/motor.stl scale=1 1 1; visual mesh filename=package://seer_description/meshes/motor.stl scale=1 1 1
Joints:
- added joint adapter_mount_joint: type fixed, parent wrist3_Link, child gripper_adapter_link, origin xyz=0 0 0 rpy=0 0 0
- added joint gripper1_joint: type prismatic, parent gripper_motor_link, child gripper1_link, origin xyz=0 0.1 -0.07 rpy=1.5707963267948966 0 0, axis 0 1 0, limit lower=0.0 upper=0.04 effort=50.0 velocity=0.1
- added joint gripper2_joint: type prismatic, parent gripper_motor_link, child gripper2_link, origin xyz=0 0.1 0.12 rpy=1.5707963267948966 3.141592653589793 0, axis 0 1 0, limit lower=0.0 upper=0.04 effort=50.0 velocity=0.1
- added joint motor_mount_joint: type fixed, parent gripper_adapter_link, child gripper_motor_link, origin xyz=-0.02 0 0.035 rpy=1.5707963267948966 0 1.5707963267948966
- joint camera_joint: origin xyz=0.00 0.08 0.00 rpy=1.5707963267948966 -1.5707963267948966 3.141592653589793 -> xyz=0.00 0.1 0.00 rpy=1.5707963267948966 -1.5707963267948966 3.141592653589793

File: seer_description/urdf/composite_robot.urdf.xacro (robot description, xacro)
@@ -13,9 +13,9 @@
       <plugin>gz_ros2_control/GazeboSimSystem</plugin>
     </hardware>
-    <xacro:macro name="aubo_joint_interface" params="joint_name">
+    <xacro:macro name="aubo_joint_interface" params="joint_name joint_min joint_max">
       <joint name="${joint_name}">
         <command_interface name="position">
-          <param name="min">-6.28</param>
-          <param name="max">6.28</param>
+          <param name="min">${joint_min}</param>
+          <param name="max">${joint_max}</param>
         </command_interface>
         <state_interface name="position" />
@@ -24,10 +24,12 @@
       </joint>
     </xacro:macro>
-    <xacro:aubo_joint_interface joint_name="shoulder_joint" />
-    <xacro:aubo_joint_interface joint_name="upperArm_joint" />
-    <xacro:aubo_joint_interface joint_name="foreArm_joint" />
-    <xacro:aubo_joint_interface joint_name="wrist1_joint" />
-    <xacro:aubo_joint_interface joint_name="wrist2_joint" />
-    <xacro:aubo_joint_interface joint_name="wrist3_joint" />
+    <xacro:aubo_joint_interface joint_name="shoulder_joint" joint_min="-6.28" joint_max="6.28" />
+    <xacro:aubo_joint_interface joint_name="upperArm_joint" joint_min="-6.28" joint_max="6.28" />
+    <xacro:aubo_joint_interface joint_name="foreArm_joint" joint_min="-6.28" joint_max="6.28" />
+    <xacro:aubo_joint_interface joint_name="wrist1_joint" joint_min="-6.28" joint_max="6.28" />
+    <xacro:aubo_joint_interface joint_name="wrist2_joint" joint_min="-6.28" joint_max="6.28" />
+    <xacro:aubo_joint_interface joint_name="wrist3_joint" joint_min="-6.28" joint_max="6.28" />
+    <xacro:aubo_joint_interface joint_name="gripper1_joint" joint_min="0.0" joint_max="0.04" />
+    <xacro:aubo_joint_interface joint_name="gripper2_joint" joint_min="0.0" joint_max="0.04" />
   </ros2_control>
   <gazebo>

Commit message: update for wo manipulator

File: seer_aubo_moveit_config/config/seer_aubo_composite.ros2_control.xacro (robot description, xacro)
@@ -50,18 +50,4 @@
                 <state_interface name="velocity"/>
             </joint>
-            <joint name="gripper1_joint">
-                <command_interface name="position"/>
-                <state_interface name="position">
-                  <param name="initial_value">${initial_positions['gripper1_joint']}</param>
-                </state_interface>
-                <state_interface name="velocity"/>
-            </joint>
-            <joint name="gripper2_joint">
-                <command_interface name="position"/>
-                <state_interface name="position">
-                  <param name="initial_value">${initial_positions['gripper2_joint']}</param>
-                </state_interface>
-                <state_interface name="velocity"/>
-            </joint>
         </ros2_control>
     </xacro:macro>
